Commit message: changes for lab 2

File: ME465_Description/urdf/robot.urdf.xacro (robot description, xacro)
@@ -88,4 +88,41 @@
     </sensor>
   </gazebo>
+  <link name="camera_link2">
+    <inertial>
+      <mass value="0.01" />
+      <origin xyz="0 0 0" />
+      <inertia ixx="0.001" ixy="0.0" ixz="0.0"
+               iyy="0.001" iyz="0.0"
+               izz="0.001" />
+    </inertial>
+  </link>
+  <joint name="camera_joint2" type="fixed">
+    <parent link="base_link"/>
+    <child link="camera_link2"/>
+    <origin rpy="0 -0.3 1.57" xyz="0 0.12 0.12"/>
+  </joint>
+  <gazebo reference="camera_link2">
+    <sensor type="camera" name="camera2">
+      <plugin name="gazebo_ros_camera_controller_2" filename="libgazebo_ros_camera.so">
+        <updateRate>0.0</updateRate>
+        <imageTopicName>image_raw2</imageTopicName>
+        <cameraInfoTopicName>camera_info2</cameraInfoTopicName>
+        <frameName>camera_link2</frameName>
+      </plugin>
+      <update_rate>30.0</update_rate>
+      <camera name="camera2">
+        <horizontal_fov>1.3962634</horizontal_fov>
+        <image>
+          <width>640</width>
+          <height>480</height>
+          <format>R8G8B8</format>
+        </image>
+        <clip>
+          <near>0.1</near>
+          <far>100</far>
+        </clip>
+      </camera>
+    </sensor>
+  </gazebo>
   <gazebo>
     <plugin name="gazebo_ros_joint_state_publisher" filename="libgazebo_ros_joint_state_publisher.so">
